File: kicad PCB files/Hepheaestes38_PCB.kicad_pcb (KiCad board)
At the start: 2 copper layers, 262.2 x 162.6 mm, 81 parts

Commit message: Added PCB Gerber Files
Parts:
- moved D18 63.4 mm to (302.4, 106.9), turned to 7 degrees
- moved S18 63.2 mm to (301.7, 102.0), turned to 7 degrees
- moved S19 63.1 mm to (299.7, 85.1), turned to 7 degrees
- moved D19 63.0 mm to (300.3, 90.0), turned to 7 degrees
- moved D1 59.7 mm to (47.9, 106.9), turned to -7 degrees
- moved S1 59.5 mm to (48.5, 102.0), turned to -7 degrees
- moved S2 59.4 mm to (50.6, 85.1), turned to -7 degrees
- moved D2 59.3 mm to (50.0, 90.0), turned to -7 degrees
- moved D20 54.8 mm to (284.4, 114.6), turned to 10 degrees
- moved S20 54.3 mm to (283.5, 109.6), turned to 10 degrees
- moved S22 53.6 mm to (277.6, 76.1), turned to 10 degrees
- moved D21 53.5 mm to (281.5, 97.8), turned to 10 degrees
- moved D22 53.4 mm to (278.5, 81.1), turned to 10 degrees
- moved S21 53.4 mm to (280.6, 92.9), turned to 10 degrees
- moved D3 51.1 mm to (65.8, 114.6), turned to -10 degrees
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Routing:
- net P5: track 13.0 -> 330.7 mm
- net P20: track 418.1 -> 623.9 mm
- net P19: track 201.2 -> 374.4 mm
- net P14: track 153.4 -> 325.9 mm
- net P16: track 127.2 -> 284.9 mm
- net P18: track 174.9 -> 318.9 mm
- net P4: track 10.8 -> 149.7 mm
- net P21: track 13.0 -> 149.5 mm
- net P15: track 155.4 -> 276.4 mm
- net GND: track 76.6 -> 162.7 mm
- net P10: track 4.32 -> 67.4 mm
- net VCC: track 32.7 -> 34.7 mm
- net P9: track 85.3 -> 84.5 mm
Other:
- board size 262.2 x 162.6 mm -> 282.3 x 119.4 mm
- rule pad_to_mask_clearance: 0.05 -> 0
