File: PCB, Case/kicad PCB files/Hepheastes38 V2 PCB/Hepheaestes38v2.kicad_pcb (KiCad board)
At the start: 2 copper layers, 282.3 x 119.4 mm, 92 parts

Commit message: Re-organised folder structure, adding v2 CAD
Parts:
- moved S31 0.24 mm to (218.0, 80.3)
- moved S28 0.24 mm to (234.7, 70.2)
- moved S38 0.24 mm to (197.0, 158.7)
- moved D5 0.24 mm to (73.5, 80.7)
- moved S22 0.24 mm to (279.4, 75.8)
- moved D33 0.24 mm to (207.0, 109.9)
- moved D37 0.24 mm to (216.7, 150.7)
- moved D9 0.24 mm to (107.0, 107.3)
- moved D36 0.24 mm to (153.3, 162.3)
- moved D2 0.24 mm to (51.7, 89.7)
- moved D17 0.24 mm to (152.8, 94.0)
- moved S32 0.24 mm to (211.3, 121.1)
- moved MH4 0.24 mm to (97.7, 111.5)
- moved D38 0.24 mm to (200.4, 162.3)
- moved B1 0.24 mm to (138.2, 132.3)
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Routing:
- net GND: track 167.6 -> 171.1 mm
- net P0: track 258.4 -> 259.5 mm
- net RAW: track 78.5 -> 77.9 mm
Other:
- board text added: "WayWayWay"

Commit message: Revised PCBv2 Gerber And files
Parts:
- moved D20 0.35 mm to (285.8, 114.3)
- moved MH7 0.35 mm to (242.6, 60.6)
- moved S22 0.35 mm to (279.1, 75.9)
- moved D9 0.35 mm to (106.7, 107.4)
- moved D6 0.35 mm to (87.4, 106.9)
- moved D18 0.35 mm to (303.8, 106.7)
- moved D22 0.35 mm to (279.9, 80.8)
- moved S13 0.35 mm to (130.1, 96.6)
- moved S36 0.35 mm to (156.4, 158.8)
- moved D24 0.35 mm to (261.3, 90.5)
- moved D10 0.35 mm to (111.9, 91.2)
- moved D5 0.35 mm to (73.1, 80.8)
- moved S34 0.35 mm to (198.8, 89.5)
- moved MH2 0.35 mm to (110.5, 60.6)
- moved MH4 0.35 mm to (97.4, 111.7)
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Connections:
- D11 pad 2: P21x -> P6
- D14 pad 2: P21x -> P6
- D17 pad 2: P21x -> P6
- D5 pad 2: P21x -> P6
- D8 pad 2: P21x -> P6
Routing:
- net P6: track 0.00 -> 185.5 mm, vias 0 -> 5
- net P21x: track 103.0 -> 0.00 mm, vias 5 -> 0
- net CS: track 38.2 -> 36.5 mm
- net GND: track 171.1 -> 170.0 mm
- net P7: track 153.3 -> 152.6 mm
Other:
- board text removed: "WayWayWay"
